Commit message: made small changes to arm_2r and added missing point at task3; completed task4.

File: week-2/.ipynb_checkpoints/arm_2r-checkpoint.urdf (robot description, URDF)
Before this commit: robot pend_robot, 6 links, 5 joints
Links:
- added link tip_link, mass 0.1; visual sphere radius=0.04
Joints:
- added joint tip_fixed: type fixed, parent arm2_link, child tip_link, origin xyz=0.6 0 0 rpy=0 0 0

File: week-2/arm_2r_EO.urdf (robot description, URDF)
Before this commit: robot pend_robot, 6 links, 5 joints
Links:
- added link tip_link, mass 0.1; visual sphere radius=0.04
Joints:
- added joint tip_fixed: type fixed, parent arm2_link, child tip_link, origin xyz=0.6 0 0 rpy=0 0 0
